Commit message: Rename some things; add an rviz file.

File: urdf/sektion_cabinet.urdf (robot description, URDF)
Before this commit: robot cabinet_sektion, 9 links, 8 joints
Links:
- link door_left_link: geometry collision mesh filename=package://sektion_cabinet_model/meshes/drawer.stl; visual mesh filename=package://sektion_cabinet_model/meshes/door.stl scale=1.0 1.0 1.0
- link door_right_link: geometry collision mesh filename=package://sektion_cabinet_model/meshes/drawer.stl; visual mesh filename=package://sektion_cabinet_model/meshes/door.stl scale=1.0 1.0 1.0
- link drawer_bottom: geometry collision mesh filename=package://sektion_cabinet_model/meshes/drawer.stl; visual mesh filename=package://sektion_cabinet_model/meshes/drawer.stl scale=1.0 1.0 1.0
- link drawer_top: geometry collision mesh filename=package://sektion_cabinet_model/meshes/drawer.stl; visual mesh filename=package://sektion_cabinet_model/meshes/drawer.stl scale=1.0 1.0 1.0
- link sektion: geometry collision mesh filename=package://sektion_cabinet_model/meshes/sektion.stl; visual mesh filename=package://sektion_cabinet_model/meshes/sektion.stl scale=1.0 1.0 1.0

Commit message: Update model and publishers to work with Lula system
- add frames centered on the doors
- publish on /tracker/tf rather than /tf (the latter is reserved for the
  robot).

File: urdf/sektion_cabinet.urdf (robot description, URDF)
Before this commit: robot cabinet_sektion, 9 links, 8 joints
Links:
- added link door_left
- added link door_right
Joints:
- added joint door_left_transform: type fixed, parent door_left_link, child door_left, origin xyz=0 .181 0 rpy=0 0 0, axis 0 0 1
- added joint door_right_transform: type fixed, parent door_right_link, child door_right, origin xyz=0 -.181 0 rpy=0 0 0, axis 0 0 1

Commit message: Improved cabinet model and URDF

File: urdf/sektion_cabinet.urdf (robot description, URDF)
Before this commit: robot cabinet_sektion, 11 links, 10 joints
Links:
- added link door_left_nob_link, mass 1.0; visual mesh filename=package://sektion_cabinet_model/meshes/door_left_nob.stl scale=1.0 1.0 1.0
- added link door_right_nob_link, mass 1.0; visual mesh filename=package://sektion_cabinet_model/meshes/door_right_nob.stl scale=1.0 1.0 1.0
- added link drawer_handle_bottom, mass 1.0; visual mesh filename=package://sektion_cabinet_model/meshes/drawer_handle.stl scale=1.0 1.0 1.0
- added link drawer_handle_top, mass 1.0; visual mesh filename=package://sektion_cabinet_model/meshes/drawer_handle.stl scale=1.0 1.0 1.0
- link door_left_link: geometry visual mesh filename=package://sektion_cabinet_model/meshes/door_left.stl scale=1.0 1.0 1.0
- link door_right_link: geometry visual mesh filename=package://sektion_cabinet_model/meshes/door_right.stl scale=1.0 1.0 1.0
- link drawer_bottom: geometry visual mesh filename=package://sektion_cabinet_model/meshes/drawer.stl scale=1.0 1.0 1.0
- link drawer_top: geometry visual mesh filename=package://sektion_cabinet_model/meshes/drawer.stl scale=1.0 1.0 1.0
- link sektion: geometry visual mesh filename=package://sektion_cabinet_model/meshes/sektion.stl scale=1.0 1.0 1.0
Joints:
- added joint door_left_nob_transform: type fixed, parent door_left_link, child door_left_nob_link, origin xyz=0 0 0 rpy=0 0 0, axis 0 0 1
- added joint door_right_nob_transform: type fixed, parent door_right_link, child door_right_nob_link, origin xyz=0 0 0 rpy=0 0 0, axis 0 0 1
- added joint drawer_handle_bottom_joint: type fixed, parent drawer_bottom, child drawer_handle_bottom, origin xyz=0 0 0 rpy=0 0 0, axis 1 0 0, limit lower=0.0 upper=0.4 effort=1000.0 velocity=0.1
- added joint drawer_handle_top_joint: type fixed, parent drawer_top, child drawer_handle_top, origin xyz=0 0 0 rpy=0 0 0, axis 1 0 0, limit lower=0.0 upper=0.4 effort=1000.0 velocity=0.1
